File: MQP Kat Foot Sensors.sch (KiCad schematic (older format))
At the start: 31 parts, among them IC1 BMP280, IC2 BMP280, IC3 BMP280, IC4 BMP280, IC5 BMP280, IC6 BMP280, IC7 BMP280, J1 Conn_01x06_Male, J2 Conn_01x04_Male, U1 STM32L432KBUx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

Commit message: updated pinout
Parts:
- removed C1, C2: 10PF, Capacitor_SMD:C_0402_1005Metric, symbol Device:C
- removed Y1: Crystal_GND24, Crystal:Crystal_SMD_2016-4Pin_2.0x1.6mm, symbol Device:Crystal_GND24
- added J3: Conn_01x04_Male, pads1x4:1x4Pads, symbol Connector:Conn_01x04_Male
Connections:
- net labels added: RX, TX
- wire segments 18 -> 15
Changed lines of the file:
@@
 $EndDescr
-$Comp
-L MCU_ST_STM32L4:STM32L432KBUx U1
-U 1 1 5B70EF37
-P 1600 3400
-F 0 "U1" H 1600 4478 50  0000 C CNN
-F 1 "STM32L432KBUx" H 1600 4387 50  0000 C CNN
-F 2 "Package_DFN_QFN:QFN-32-1EP_5x5mm_P0.5mm_EP3.45x3.45mm" H 1200 2500 50  0001 R CNN
-F 3 "http://www.st.com/st-web-ui/static/active/en/resource/technical/document/datasheet/DM00257205.pdf" H 1600 3400 50  0001 C CNN
-	1    1600 3400
-	1    0    0    -1
-$EndComp
 $Comp
 L Connector:Conn_01x04_Male J2
@@
 	1    0    0    -1
 $EndComp
-Text GLabel 3600 5350 0    50   Input ~ 0
+Text GLabel 3650 6750 0    50   Input ~ 0
 CS5
 Text GLabel 3600 5450 0    50   Input ~ 0
@@
 	1    1600 4400
 	1    0    0    -1
-$EndComp
-Wire Wire Line
-	750  3200 1100 3200
-Wire Wire Line
-	1100 3200 1100 3300
-Wire Wire Line
-	750  3500 1100 3500
-Wire Wire Line
-	1100 3500 1100 3400
-$Comp
-L power:GND #PWR0136
-U 1 1 5B7109DC
-P 950 3350
-F 0 "#PWR0136" H 950 3100 50  0001 C CNN
-F 1 "GND" V 955 3222 50  0000 R CNN
-F 2 "" H 950 3350 50  0001 C CNN
-F 3 "" H 950 3350 50  0001 C CNN
-	1    950  3350
-	0    -1   -1   0
-$EndComp
-$Comp
-L power:GND #PWR0137
-U 1 1 5B710A70
-P 550 3350
-F 0 "#PWR0137" H 550 3100 50  0001 C CNN
-F 1 "GND" V 555 3222 50  0000 R CNN
-F 2 "" H 550 3350 50  0001 C CNN
-F 3 "" H 550 3350 50  0001 C CNN
-	1    550  3350
-	0    1    1    0
 $EndComp
 Text GLabel 2100 3300 2    50   Input ~ 0
@@
 $EndComp
 $Comp
-L Device:C C1
-U 1 1 5B711078
-P 750 3050
-F 0 "C1" H 865 3096 50  0000 L CNN
-F 1 "10PF" H 865 3005 50  0000 L CNN
-F 2 "Capacitor_SMD:C_0402_1005Metric" H 788 2900 50  0001 C CNN
-F 3 "~" H 750 3050 50  0001 C CNN
-	1    750  3050
-	1    0    0    -1
-$EndComp
-$Comp
-L Device:C C2
-U 1 1 5B7110FF
-P 750 3650
-F 0 "C2" H 865 3696 50  0000 L CNN
-F 1 "10PF" H 865 3605 50  0000 L CNN
-F 2 "Capacitor_SMD:C_0402_1005Metric" H 788 3500 50  0001 C CNN
-F 3 "~" H 750 3650 50  0001 C CNN
-	1    750  3650
-	1    0    0    -1
-$EndComp
-$Comp
-L power:GND #PWR0138
-U 1 1 5B711169
-P 750 3800
-F 0 "#PWR0138" H 750 3550 50  0001 C CNN
-F 1 "GND" H 755 3627 50  0000 C CNN
-F 2 "" H 750 3800 50  0001 C CNN
-F 3 "" H 750 3800 50  0001 C CNN
-	1    750  3800
-	1    0    0    -1
-$EndComp
-$Comp
-L power:GND #PWR0139
-U 1 1 5B7111CD
-P 750 2900
-F 0 "#PWR0139" H 750 2650 50  0001 C CNN
-F 1 "GND" H 755 2727 50  0000 C CNN
-F 2 "" H 750 2900 50  0001 C CNN
-F 3 "" H 750 2900 50  0001 C CNN
-	1    750  2900
-	-1   0    0    1
-$EndComp
-$Comp
 L power:GND #PWR0140
 U 1 1 5B7112E8
@@
 	1    0    0    -1
 $EndComp
-Text GLabel 3650 6750 0    50   Input ~ 0
+Text GLabel 3600 5350 0    50   Input ~ 0
 CS6
 Text GLabel 5850 5450 0    50   Input ~ 0
@@
 Text GLabel 2100 3000 2    50   Input ~ 0
 CS7
-Text GLabel 2100 3800 2    50   Input ~ 0
+Text GLabel 1100 3900 0    50   Input ~ 0
 MISO2
-Text GLabel 2100 3900 2    50   Input ~ 0
+Text GLabel 1100 4000 0    50   Input ~ 0
 MOSI2
 Text GLabel 1100 3800 0    50   Input ~ 0
 SCK2
-$Comp
-L Device:Crystal_GND24 Y1
-U 1 1 5B809917
-P 750 3350
-F 0 "Y1" V 704 3591 50  0000 L CNN
-F 1 "Crystal_GND24" V 795 3591 50  0000 L CNN
-F 2 "Crystal:Crystal_SMD_2016-4Pin_2.0x1.6mm" H 750 3350 50  0001 C CNN
-F 3 "~" H 750 3350 50  0001 C CNN
-	1    750  3350
-	0    1    1    0
-$EndComp
-Connection ~ 750  3200
-Connection ~ 750  3500
 $Comp
 L power:+BATT #PWR0158
@@
 $EndComp
 $Comp
-L power:GND #PWR0160
-U 1 1 5B80AD7A
-P 4250 1550
-F 0 "#PWR0160" H 4250 1300 50  0001 C CNN
-F 1 "GND" V 4255 1422 50  0000 R CNN
-F 2 "" H 4250 1550 50  0001 C CNN
-F 3 "" H 4250 1550 50  0001 C CNN
-	1    4250 1550
-	0    1    1    0
-$EndComp
-$Comp
 L power:GND #PWR0161
 U 1 1 5B80AE10
@@
 	-1   0    0    1
 $EndComp
+$Comp
+L MCU_ST_STM32L4:STM32L432KBUx U1
+U 1 1 5B70EF37
+P 1600 3400
+F 0 "U1" H 1600 4478 50  0000 C CNN
+F 1 "STM32L432KBUx" H 1600 4387 50  0000 C CNN
+F 2 "Package_DFN_QFN:QFN-32-1EP_5x5mm_P0.5mm_EP3.45x3.45mm" H 1200 2500 50  0001 R CNN
+F 3 "http://www.st.com/st-web-ui/static/active/en/resource/technical/document/datasheet/DM00257205.pdf" H 1600 3400 50  0001 C CNN
+	1    1600 3400
+	1    0    0    -1
+$EndComp
+Wire Wire Line
+	4250 1350 4250 1550
+$Comp
+L power:+3.3V #PWR0136
+U 1 1 5BAD5B11
+P 2450 2000
+F 0 "#PWR0136" H 2450 1850 50  0001 C CNN
+F 1 "+3.3V" H 2465 2173 50  0000 C CNN
+F 2 "" H 2450 2000 50  0001 C CNN
+F 3 "" H 2450 2000 50  0001 C CNN
+	1    2450 2000
+	-1   0    0    1
+$EndComp
+$Comp
+L power:GND #PWR0137
+U 1 1 5BAD5B5C
+P 2550 2000
+F 0 "#PWR0137" H 2550 1750 50  0001 C CNN
+F 1 "GND" H 2555 1827 50  0000 C CNN
+F 2 "" H 2550 2000 50  0001 C CNN
+F 3 "" H 2550 2000 50  0001 C CNN
+	1    2550 2000
+	1    0    0    -1
+$EndComp
+Text GLabel 2650 2000 3    50   Input ~ 0
+TX
+Text GLabel 2750 2000 3    50   Input ~ 0
+RX
+Text GLabel 1100 4200 0    50   Input ~ 0
+RX
+Text GLabel 2100 3600 2    50   Input ~ 0
+TX
+$Comp
+L Connector:Conn_01x04_Male J3
+U 1 1 5BAD6448
+P 2650 1800
+F 0 "J3" V 2710 1940 50  0000 L CNN
+F 1 "Conn_01x04_Male" V 2801 1940 50  0000 L CNN
+F 2 "pads1x4:1x4Pads" H 2650 1800 50  0001 C CNN
+F 3 "~" H 2650 1800 50  0001 C CNN
+	1    2650 1800
+	0    1    1    0
+$EndComp
 $EndSCHEMATC
